File: pcb/solar-board/solar.kicad_sch (KiCad schematic)
At the start: 201 parts, among them J1 XT30_panelA, J2 XT30_panelB, J3 XT60_battery, J4 XT60_ESCout, J5 JST-XH_balance, J6 JST-GH_toFC, J7 JST-GH_I2C, J8 USB_C_Receptacle_USB2.0_16P, J9 JST-PH_servo, Q1 SIR626DP, Q10 Q_NMOS_GSD, Q11 Q_NMOS_GSD, Q12 Q_NMOS_GSD, Q2 SIR626DP, Q3 SIR626DP, Q4 SIR626DP, Q5 SIR626DP, Q6 SIR626DP, Q7 SIR626DP, Q8 SIR626DP, Q9 Q_NMOS_GSD, SW1 tact, U1 LM5175RHFR, U10 TPS54302DDCR, U11 AP2112K-3.3TRG1, U12 ESP32-C3-MINI-1-N4, U13 MCP4728A0T-E_UN, U2 LM5175RHFR, U3 INA228AIDGSR, U4 INA228AIDGSR, U5 INA228AIDGSR, U6 BQ7692000PWR, U7 TLV9061IDCKR, U8 TLV9061IDCKR, U9 TPS54202DDCR

Commit message: pcb
Parts:
- Q1, Q2, Q3, Q4, Q5, Q6, Q7, Q8: footprint SIR626DP_T1_RE3:MOSFET_DP-T1-RE3_VIS -> Package_SO:PowerPAK_SO-8_Single
Other:
- moved on the sheet: C1, C10, C11, C12, C13, C14, C15, C16, C17, C18, C19, C2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
