File: pcb/solar-board/solar.kicad_pcb (KiCad board)
At the start: 2 copper layers, 149.6 x 65 mm, 201 parts, among them J1 XT30_panelA, J2 XT30_panelB, J3 XT60_battery, J4 XT60_ESCout, J5 JST-XH_balance, J6 JST-GH_toFC, J7 JST-GH_I2C, J8 USB_C_Receptacle_USB2.0_16P, J9 JST-PH_servo, Q1 SIR626DP, Q10 Q_NMOS_GSD, Q11 Q_NMOS_GSD, Q12 Q_NMOS_GSD, Q2 SIR626DP, Q3 SIR626DP, Q4 SIR626DP, Q5 SIR626DP, Q6 SIR626DP, Q7 SIR626DP, Q8 SIR626DP, Q9 Q_NMOS_GSD, SW1 tact, U1 LM5175RHFR, U10 TPS54302DDCR, U11 AP2112K-3.3TRG1, U12 ESP32-C3-MINI-1-N4, U13 MCP4728A0T-E_UN, U2 LM5175RHFR, U3 INA228AIDGSR, U4 INA228AIDGSR, U5 INA228AIDGSR, U6 BQ7692000PWR, U7 TLV9061IDCKR, U8 TLV9061IDCKR, U9 TPS54202DDCR

Commit message: pcb
Parts:
- moved U12 746.9 mm to (143.4, 110.5), turned to 180 degrees
- moved C88 736.1 mm to (152.8, 104.0)
- moved C85 731.6 mm to (121.0, 101.8), turned to -90 degrees
- moved U13 730.4 mm to (142.0, 95.0), turned to 90 degrees
- moved R70 729.9 mm to (153.2, 108.5), turned to -90 degrees
- moved C86 724.4 mm to (112.3, 100.0), turned to 180 degrees
- moved R60 722.7 mm to (149.0, 97.3), turned to 90 degrees
- moved R72 722.3 mm to (153.0, 105.7)
- moved R61 719.8 mm to (147.0, 97.3), turned to 90 degrees
- moved C87 718.4 mm to (112.2, 96.9), turned to 180 degrees
- moved R75 713.8 mm to (127.0, 110.2), turned to 90 degrees
- moved R71 713.5 mm to (138.0, 97.6), turned to 90 degrees
- moved R76 711.8 mm to (129.0, 110.2), turned to 90 degrees
- moved C92 710.4 mm to (112.2, 93.5), turned to 180 degrees
- moved R73 709.8 mm to (145.0, 97.3), turned to 90 degrees
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Routing:
- net /+3V3: track 0.00 -> 169.1 mm, vias 0 -> 6
- net /BMS_ALERT: track 0.00 -> 163.6 mm, vias 0 -> 5
- net /SCL: track 0.00 -> 127.9 mm, vias 0 -> 6
- net /PACK_P: track 0.00 -> 126.2 mm, vias 0 -> 2
- net /SDA: track 0.00 -> 120.9 mm, vias 0 -> 2
- net /VPACK: track 65.5 -> 169.6 mm, vias 4 -> 6
- net /EN_A_CTL: track 0.00 -> 99.0 mm, vias 0 -> 2
- net /SW1_B: track 0.00 -> 96.2 mm, vias 0 -> 2
- net /VIN_B: track 0.00 -> 83.2 mm, vias 0 -> 2
- net /DAC_MPPT_A: track 0.00 -> 68.5 mm, vias 0 -> 2
- net /VIN_A: track 78.8 -> 146.3 mm
- net /DAC_MPPT_B: track 0.00 -> 57.5 mm, vias 0 -> 3
- net /SOL_A_P: track 25.0 -> 81.1 mm
- net /SOL_B_P: track 0.00 -> 54.3 mm, vias 0 -> 2
- net /CSP_B: track 0.00 -> 47.9 mm
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
Commit message: pcb
Routing:
- net /VPACK: track 169.6 -> 274.4 mm, vias 6 -> 12
- net /DAC_CV_A: track 0.00 -> 68.7 mm, vias 0 -> 4
- net /+3V3: track 169.1 -> 236.2 mm, vias 6 -> 14
- net /DAC_CV_B: track 0.00 -> 48.2 mm, vias 0 -> 6
- net /+5V: track 32.7 -> 66.2 mm, vias 0 -> 2
- net /SW2_B: track 18.3 -> 41.4 mm, vias 0 -> 5

Commit message: pcb
Routing:
- net /PGND: track 0.00 -> 382.4 mm, vias 0 -> 31
- net /AGND: track 0.00 -> 271.5 mm, vias 0 -> 37
- net /FB_B: track 13.6 -> 23.8 mm
- net /DAC_MPPT_B: track 57.5 -> 66.3 mm, vias 3 -> 4
- net /USB_DP: vias 2 -> 1
- net /USB_CC2: vias 2 -> 1
- net /SW2_B: vias 5 -> 4
- added copper zone on B.Cu, net /AGND
- added copper zone on B.Cu, net /PGND

Commit message: pcb
Routing:
- net /AGND: track 271.5 -> 455.7 mm, vias 37 -> 49
- net /PGND: track 382.4 -> 468.7 mm, vias 31 -> 45
- net /SW1_A: track 19.3 -> 41.8 mm, vias 0 -> 2
- net /VIN_A: track 146.3 -> 153.0 mm, vias 0 -> 2
- net /PACK_P: track 126.2 -> 128.2 mm

Commit message: pcb
Parts:
- moved C64 0.13 mm to (179.2, 56.0)
Routing:
- net /PGND: track 468.7 -> 484.3 mm, vias 45 -> 46
Changed lines of the file:
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@@
 	(footprint "Capacitor_SMD:C_0603_1608Metric"
 		(layer "F.Cu")
-		(at 179.237498 55.874997)
+		(at 179.237498 56)
 		(descr "Capacitor SMD 0603 (1608 Metric), square (rectangular) end terminal, IPC-7351 nominal, (Body size source: IPC-SM-782 page 76, https://www.pcb-3d.com/wordpress/wp-content/uploads/ipc-sm-782a_amendment_1_and_2.pdf)")
 		(tags "capacitor")
@@
 	)
 	(via
-		(at 168.7 81.46)
+		(at 85 93.350001)
 		(size 0.6)
 		(drill 0.3)
@@
 	)
 	(via
-		(at 85 93.350001)
+		(at 188.747596 111)
 		(size 0.6)
 		(drill 0.3)
@@
 	)
 	(via
-		(at 188.747596 111)
+		(at 125 99)
 		(size 0.6)
 		(drill 0.3)
@@
 	)
 	(via
-		(at 125 99)
+		(at 168.7 81)
 		(size 0.6)
 		(drill 0.3)
@@
 	)
 	(segment
-		(start 136.5 88.792893)
-		(end 136.792893 88.5)
+		(start 171.262628 81.46)
+		(end 169.16 81.46)
 		(width 0.2)
 		(layer "B.Cu")
@@
 	)
 	(segment
-		(start 83 72)
-		(end 81 70)
+		(start 136.5 88.792893)
+		(end 136.792893 88.5)
 		(width 0.2)
 		(layer "B.Cu")
@@
 	)
 	(segment
-		(start 171.262628 81.46)
-		(end 168.7 81.46)
+		(start 83 72)
+		(end 81 70)
 		(width 0.2)
 		(layer "B.Cu")
@@
 	)
 	(segment
+		(start 169.16 81.46)
+		(end 168.7 81)
+		(width 0.2)
+		(layer "B.Cu")
+		(net "/AGND")
+	)
+	(segment
 		(start 180 93)
 		(end 177.3 93)
@@
 	)
 	(segment
+		(start 161.3 57.46)
+		(end 161.3 57.5)
+		(width 0.2)
+		(layer "F.Cu")
+		(net "/VPACK")
+	)
+	(segment
 		(start 162 111)
 		(end 162 108)
@@
 	)
 	(via
+		(at 161.3 57.46)
+		(size 0.6)
+		(drill 0.3)
+		(layers "F.Cu" "B.Cu")
+		(net "/VPACK")
+	)
+	(via
 		(at 85.8 95.65)
 		(size 0.6)
@@
 	)
 	(via
-		(at 161.3 57.36)
-		(size 0.6)
-		(drill 0.3)
-		(layers "F.Cu" "B.Cu")
-		(net "/VPACK")
-	)
-	(via
 		(at 160 78)
 		(size 0.6)
@@
 	(segment
 		(start 160.6 58.06)
-		(end 161.3 57.36)
+		(end 160.7 58.06)
+		(width 0.2)
+		(layer "B.Cu")
+		(net "/VPACK")
+	)
+	(segment
+		(start 160.7 58.06)
+		(end 161.3 57.46)
 		(width 0.2)
 		(layer "B.Cu")
@@
 	)
 	(segment
-		(start 68.05 84)
-		(end 69.05 83)
-		(width 0.2)
-		(layer "F.Cu")
-		(net "/PGND")
-	)
-	(segment
 		(start 202.696226 85)
 		(end 202 85)
@@
 	)
 	(segment
+		(start 90.5 116.5)
+		(end 100 116.5)
+		(width 0.2)
+		(layer "F.Cu")
+		(net "/PGND")
+	)
+	(segment
 		(start 171.325001 56.325)
 		(end 172.821446 57.821445)
@@
 	)
 	(segment
-		(start 68.05 87)
-		(end 68.05 84)
-		(width 0.2)
-		(layer "F.Cu")
-		(net "/PGND")
-	)
-	(segment
 		(start 128.45 67.503774)
 		(end 128.45 68)
@@
 	)
 	(segment
+		(start 89 111)
+		(end 89 115)
+		(width 0.2)
+		(layer "F.Cu")
+		(net "/PGND")
+	)
+	(segment
 		(start 188.7 104)
 		(end 191 106.3)
@@
 	)
 	(segment
+		(start 69.05 83)
+		(end 68.05 84)
+		(width 0.2)
+		(layer "F.Cu")
+		(net "/PGND")
+	)
+	(segment
 		(start 205.55 73)
 		(end 205.55 64.35)
@@
 	)
 	(segment
+		(start 68.05 84)
+		(end 68.05 87)
+		(width 0.2)
+		(layer "F.Cu")
+		(net "/PGND")
+	)
+	(segment
 		(start 159.05 100)
 		(end 159.707107 100)
@@
 	)
 	(segment
+		(start 89 115)
+		(end 90.5 116.5)
+		(width 0.2)
+		(layer "F.Cu")
+		(net "/PGND")
+	)
+	(segment
 		(start 185.4516 93.187059)
 		(end 185.4516 91.951599)
@@
 	)
 	(via
+		(at 100 116.5)
+		(size 0.6)
+		(drill 0.3)
+		(layers "F.Cu" "B.Cu")
+		(net "/PGND")
+	)
+	(via
 		(at 166 74)
 		(size 0.6)
@@
 	)
 	(via
+		(at 69.05 83)
+		(size 0.6)
+		(drill 0.3)
+		(layers "F.Cu" "B.Cu")
+		(net "/PGND")
+	)
+	(via
 		(at 102 85)
 		(size 0.6)
@@
 	)
 	(via
-		(at 69.025 83.025)
-		(size 0.6)
-		(drill 0.3)
-		(layers "F.Cu" "B.Cu")
-		(net "/PGND")
-	)
-	(via
 		(at 172.821446 57.821445)
 		(size 0.6)
@@
 	)
 	(segment
-		(start 182 60.149998)
-		(end 180.394999 60.149998)
+		(start 181.874997 57.862499)
+		(end 180.012498 56)
 		(width 0.2)
 		(layer "F.Cu")
@@
 	)
 	(segment
-		(start 180.012498 55.874997)
-		(end 182 57.862499)
+		(start 182 60.149998)
+		(end 180.394999 60.149998)
 		(width 0.2)
 		(layer "F.Cu")
@@
 	)
 	(segment
+		(start 182 57.862499)
+		(end 181.874997 57.862499)
+		(width 0.2)
+		(layer "F.Cu")
+		(net "/CELL1")
+	)
+	(segment
 		(start 185.5 66.5)
 		(end 184 68)
@@
 	)
 	(segment
-		(start 178.462498 55.874997)
-		(end 178.462498 57.862497)
+		(start 178.449998 57.874997)
+		(end 178.449998 56.0125)
 		(width 0.2)
 		(layer "F.Cu")
@@
 		(width 0.2)
 		(layer "F.Cu")
+		(net "/VC0")
+	)
+	(segment
+		(start 178.449998 56.0125)
+		(end 178.462498 56)
+		(width 0.2)
+		(layer "F.Cu")
