File: pcb/flight-controller/flight-controller.kicad_sch (KiCad schematic)
At the start: 0 parts

Commit message: flight controller
Other:
- added sheet 01_POWER (01_power.kicad_sch)
- added sheet 02_MCU (02_mcu.kicad_sch)
- added sheet 03_SENSORS (03_sensors.kicad_sch)
- added sheet 04_ACTUATORS (04_actuators.kicad_sch)
- added sheet 05_WINCH (05_winch.kicad_sch)
- added sheet 06_COMMS_IO (06_comms_io.kicad_sch)
