File: pcb/flight-controller/flight-controller.kicad_pcb (KiCad board)
At the start: 2 copper layers, 149 x 65 mm, 155 parts, among them J101 XT60_PACK_IN, J102 XT60_ESC_OUT, J201 USB-C, J202 SWD+SWO, J401 ESC_SIGNAL, J402 SERVO1_AIL_L, J403 SERVO2_AIL_R, J404 SERVO3_ELEVATOR, J405 SERVO4_RUDDER, J501 N20_1, J502 N20_2, J503 N20_3, J504 N20_4, J601 GPS_COMPASS, J602 RC_IN_CRSF_SBUS, J603 TELEM1_MAVLINK, J604 SOLAR_BOARD_J6, J605 I2C_AIRSPEED, J606 UART5_SPARE, J607 SAFETY_SWITCH, J608 ANALOG_IN, Q601 2N7002, Q602 2N7002, SW201 RESET, SW202 BOOT0/DFU, U101 INA228AIDGSR, U102 TPS54202DDCR, U103 TPS54302DDCR, U104 TPS54302DDCR, U105 AP2112K-3.3TRG1, U201 STM32F405RGT6, U202 USBLC6-2SC6, U301 ICM-42688-P, U302 DPS310XTSA1, U303 W25Q128JVSIQ, U501 DRV8833PWP, U502 DRV8833PWP, Y201 8.000MHz 10ppm CL8pF

Commit message: change connector directions
Parts:
- moved J101 6.21 mm to (7.90, 4.15), turned to 90 degrees
- moved J102 4.75 mm to (7.75, 53.3), turned to 90 degrees
- moved J201 4.53 mm to (142.9, 8.40), turned to 90 degrees
- moved U101 4.46 mm to (3.75, 19.0)
- moved D102 3.45 mm to (18.2, 14.2)
Routing:
- net VBUS: track 179.4 -> 165.8 mm
- net /01_POWER/LDO_IN: track 31.7 -> 41.2 mm, vias 0 -> 3
- net /02_MCU/USB_CC2: track 29.5 -> 24.5 mm, vias 1 -> 0
- net /02_MCU/USB_CC1: track 24.2 -> 19.4 mm, vias 1 -> 0
- net +5V: track 262.3 -> 257.8 mm, vias 3 -> 4
- net /01_POWER/VPACK: track 68.1 -> 63.7 mm, vias 2 -> 6
- net I2C2_SDA: track 211.1 -> 215.5 mm
- net /01_POWER/VBATT_IN: track 41.5 -> 45.7 mm, vias 2 -> 4
- net +3V3: track 463.6 -> 459.7 mm
- net /02_MCU/USB_DP: track 55.4 -> 52.5 mm
- net /02_MCU/USB_DM: track 68.8 -> 67.8 mm
- net GNDPWR: vias 286 -> 279
